File: eda/astable_dev/astable_dev.kicad_pcb (KiCad board)
At the start: 2 copper layers, 0 parts

Commit message: dev board complete
Parts:
- added BT1: CR2032 3V, 0_local:BatteryHolder_CR2032-BS-2-1_Front_backsilk, F.Cu at (122.4, 83.1)
- added C1: 100 uF, 0_local:CP_Radial_D5.0mm_P2.00mm_backsilk, F.Cu at (139.7, 105.4)
- added C2: 100 uF, 0_local:CP_Radial_D5.0mm_P2.00mm_backsilk, F.Cu at (127.0, 105.4)
- added D1: LED, 0_local:LED_D3.0mm-2_backsilk, F.Cu at (151.1, 113.0)
- added D2: LED, 0_local:LED_D3.0mm-2_backsilk, F.Cu at (115.6, 113.0)
- added G***: LOGO, 0_alt_bier:logo-alt_bier-1200dpi-8x19mm-front, F.Cu at (150.4, 81.5)
- added GND: Test Point GND1, 0_local:Conn_Pin_Header_Hole_1x01_Pitch2.54mm, F.Cu at (133.3, 111.8)
- added Q1: 2N2222A, 0_local:Q_2222A_TO-92_Inline_back-silk, F.Cu at (142.2, 113.0)
- added Q2: 2N2222A, 0_local:Q_2222A_TO-92_Inline_back-silk, F.Cu at (124.5, 113.0)
- added R1: 1K Ohms, 0_local:R_Axial_DIN0204_L3.6mm_D1.6mm_P5.08mm_Horizontal_backsilk, F.Cu at (137.2, 95.2)
- added R2: 1K Ohms, 0_local:R_Axial_DIN0204_L3.6mm_D1.6mm_P5.08mm_Horizontal_backsilk, F.Cu at (129.5, 100.3)
- added R3: 510 Ohms, 0_local:R_Axial_DIN0204_L3.6mm_D1.6mm_P5.08mm_Horizontal_backsilk, F.Cu at (148.6, 104.1)
- added R4: 510 Ohms, 0_local:R_Axial_DIN0204_L3.6mm_D1.6mm_P5.08mm_Horizontal_backsilk, F.Cu at (123.2, 104.1)
- added R5: 10 Ohms, 0_local:R_Axial_DIN0204_L3.6mm_D1.6mm_P5.08mm_Horizontal_backsilk, F.Cu at (148.6, 106.7)
- added R6: 10 Ohms, 0_local:R_Axial_DIN0204_L3.6mm_D1.6mm_P5.08mm_Horizontal_backsilk, F.Cu at (123.2, 106.7)
- added RV1: 0-30K Ohms, 0_local:R_Potentiometer_3pin_THT_5mm_backsilk_anno, F.Cu at (148.6, 94.0)
- added RV2: 0-30K Ohms, 0_local:R_Potentiometer_3pin_THT_5mm_backsilk_anno, F.Cu at (123.2, 94.0)
- added TP1: Test Point 1, 0_local:Conn_Pin_Header_Hole_1x01_Pitch2.54mm, F.Cu at (151.1, 106.7)
- added TP2: Test Point 2, 0_local:Conn_Pin_Header_Hole_1x01_Pitch2.54mm, F.Cu at (115.6, 106.7)
- added TP3: Test Point 3, 0_local:Conn_Pin_Header_Hole_1x01_Pitch2.54mm, F.Cu at (137.2, 111.8)
- added TP4: Test Point 4, 0_local:Conn_Pin_Header_Hole_1x01_Pitch2.54mm, F.Cu at (129.5, 111.8)
- added TPJ1: Test Point Connector, 0_local:Conn_Pin_Header_Hole_1x05_Pitch2.54mm, F.Cu at (115.6, 80.3)
Routing:
- net TP3: track 0.00 -> 92.8 mm
- net TP4: track 0.00 -> 74.5 mm
- net TP1: track 0.00 -> 67.0 mm
- net Net-(BT1-Pad1): track 0.00 -> 63.3 mm
- net TP2: track 0.00 -> 31.9 mm
- net GND: track 0.00 -> 18.3 mm
- net Net-(C2-Pad1): track 0.00 -> 11.2 mm
- net Net-(C1-Pad1): track 0.00 -> 11.2 mm
- net Net-(R1-Pad1): track 0.00 -> 10.5 mm
- net Net-(R2-Pad2): track 0.00 -> 10.4 mm
- added copper zone on B.Cu, net GND
Other:
- board outline added: 43.2 x 45 mm
- board text added: "0-30kR"
- board text added: "100uF"
- board text added: "10R"
- board text added: "1kR"
- board text added: "510R"
- board text added: "Astable"
- board text added: "GND"
- board text added: "LED"
- board text added: "Multivibrator"
- board text added: "Place Coin Cell Battery With + Side Up"
- board text added: "TP1"
- board text added: "TP2"
- board text added: "TP3"
- board text added: "TP4"
