File: eda/astable_badge/astable_badge.kicad_pcb (KiCad board)
At the start: 2 copper layers, 0 parts

Commit message: Final badge art and EDA updates.
Parts:
- added BT1: CR2032 3V, 0_local:BatteryHolder_CR2032-BS-2-1_Front_backsilk, F.Cu at (192.3, 124.7)
- added C1: 100 uF, 0_local:CP_Radial_D5.0mm_P2.00mm_backsilk, F.Cu at (121.4, 61.3)
- added C2: 100 uF, 0_local:CP_Radial_D5.0mm_P2.00mm_backsilk, F.Cu at (126.9, 64.1)
- added D1: LED, 0_local:LED_D3.0mm-2_backsilk, F.Cu at (139.1, 37.1)
- added D2: LED, 0_local:LED_D3.0mm-2_backsilk, F.Cu at (146.7, 37.1)
- added G***: LOGO, 0_local:2021, F.Cu at (149.9, 120.1)
- added G***: LOGO, 0_alt_bier:logo-alt_bier-700dpi-13x32mm-back, F.Cu at (180.1, 85.1)
- added G***: LOGO, 0_org_logos:BSidesDFW_Logo_Front_900dpi, F.Cu at (135.8, 140.2)
- added G***: LOGO, 0_local:CyberDolphin1_500dpi_108mm, F.Cu at (143.6, 78.9)
- added Q1: 2N2222A, 0_local:Q_2222A_TO-92_Inline_back-silk, F.Cu at (116.1, 66.1)
- added Q2: 2N2222A, 0_local:Q_2222A_TO-92_Inline_back-silk, F.Cu at (129.5, 71.5)
- added R1: 1K R, 0_local:R_Axial_DIN0204_L3.6mm_D1.6mm_P5.08mm_Horizontal_backsilk, F.Cu at (129.8, 47.4)
- added R2: 1K R, 0_local:R_Axial_DIN0204_L3.6mm_D1.6mm_P5.08mm_Horizontal_backsilk, F.Cu at (151.4, 44.8)
- added R3: 510 R, 0_local:R_Axial_DIN0204_L3.6mm_D1.6mm_P5.08mm_Horizontal_backsilk, F.Cu at (131.6, 48.1)
- added R4: 510 R, 0_local:R_Axial_DIN0204_L3.6mm_D1.6mm_P5.08mm_Horizontal_backsilk, F.Cu at (149.4, 45.6)
- added R5: 10 R, 0_local:R_Axial_DIN0204_L3.6mm_D1.6mm_P5.08mm_Horizontal_backsilk, F.Cu at (129.4, 44.8)
- added R6: 10 R, 0_local:R_Axial_DIN0204_L3.6mm_D1.6mm_P5.08mm_Horizontal_backsilk, F.Cu at (147.3, 50.6)
- added REF**: Astable_Multivibrator_Circuit, 0_local:Astable_Multivibrator_Circuit-back, F.Cu at (131.3, 105.4)
- added RV1: 0-30K Ohms, 0_local:R_Potentiometer_3pin_THT_5mm_backsilk_anno, F.Cu at (120.6, 53.6)
- added RV2: 0-30K Ohms, 0_local:R_Potentiometer_3pin_THT_5mm_backsilk_anno, F.Cu at (158.5, 51.9)
- added TPJ1: Test Point Connector, 0_local:Conn_Pin_Header_Hole_1x05_Pitch2.54mm, F.Cu at (176.0, 111.3)
Routing:
- net GND: track 0.00 -> 201.8 mm
- net TP2: track 0.00 -> 166.0 mm
- net TP3: track 0.00 -> 137.0 mm
- net TP1: track 0.00 -> 133.2 mm
- net Net-(BT1-Pad1): track 0.00 -> 132.0 mm
- net TP4: track 0.00 -> 130.2 mm
- net Net-(C2-Pad1): track 0.00 -> 47.3 mm
- net Net-(C1-Pad1): track 0.00 -> 31.2 mm
- net Net-(R1-Pad1): track 0.00 -> 6.22 mm
- net Net-(R2-Pad2): track 0.00 -> 4.82 mm
Other:
- board outline added: 108.2 x 137.9 mm
- board text added: "Astable Multivibrator Circuit Schematic"
- board text added: "GND"
- board text added: "TP1"
- board text added: "TP2"
- board text added: "TP3"
- board text added: "TP4"
- board text added: "“We're an information economy. They teach you that in school. What they don't tell you is that it's impossible to move, to live, to operate at any level without leaving traces, bits, seemingly meaningless fragments of personal information. Fragments that can be retrieved, amplified...” ― William Gibson, author of Johnny Mnemonic"
